Commit message: front rear wheel driver

File: description/ros2_control/hoverboard_driver.ros2_control.xacro (robot description, xacro)
@@ -1,5 +1,5 @@
 <?xml version="1.0"?>
 <robot xmlns:xacro="http://www.ros.org/wiki/xacro">
-  <xacro:macro name="hoverboard_driver_ros2_control" params="name prefix">
+  <xacro:macro name="hoverboard_driver_ros2_control" params="name prefix device">
     <ros2_control name="${name}" type="system">
       <hardware>
@@ -7,6 +7,5 @@
         <param name="wheel_radius">0.0825</param>
         <param name="max_velocity">1.0</param>
-        <!-- <param name="device">/dev/ttyV1</param> -->
-        <param name="device">/dev/ttyUSB0</param>
+        <param name="device">${device}</param>
       </hardware>
       <joint name="${prefix}left_wheel_joint">

File: description/urdf/diffbot.urdf.xacro (robot description, xacro)
@@ -9,5 +9,5 @@
   <xacro:include filename="$(find hoverboard_driver)/ros2_control/hoverboard_driver.ros2_control.xacro"/>
   <xacro:diffbot prefix="$(arg prefix)" />
-  <xacro:hoverboard_driver_ros2_control
-    name="DiffBot" prefix="$(arg prefix)" />
+  <xacro:hoverboard_driver_ros2_control name="front_hoverboard" prefix="front_" device="/dev/ttyUSB0"/>
+  <xacro:hoverboard_driver_ros2_control name="rear_hoverboard" prefix="rear_" device="/dev/ttyUSB1"/>
 </robot>

File: description/urdf/diffbot_description.urdf.xacro (robot description, xacro)
@@ -55,40 +55,4 @@
         <material>Gazebo/White</material>
     </gazebo>
-    <!-- virtual left wheel -->
-    <link name="${prefix}left_wheel">
-      <visual>
-        <origin xyz="0 0 0" rpy="${PI/2} 0 ${PI/2}"/>
-        <geometry>
-          <cylinder length="0.01" radius="${wheel_radius}"/>
-        </geometry>
-        <material name="invisible"/>
-      </visual>
-    </link>
-    <joint name="${prefix}left_wheel_joint" type="continuous">
-      <parent link="${prefix}chassis_link"/>
-      <child link="${prefix}left_wheel"/>
-      <origin xyz="0 -${base_width/2} -${base_height/2}" rpy="0 0 ${PI/2}"/>
-      <axis xyz="1 0 0"/>
-      <limit effort="100.0" velocity="1.0"/>
-      <dynamics damping="0.2"/>
-    </joint>
-    <!-- virtual right wheel -->
-    <link name="${prefix}right_wheel">
-      <visual>
-        <origin xyz="0 0 0" rpy="${PI/2} 0 ${PI/2}"/>
-        <geometry>
-          <cylinder length="0.01" radius="${wheel_radius}"/>
-        </geometry>
-        <material name="invisible"/>
-      </visual>
-    </link>
-    <joint name="${prefix}right_wheel_joint" type="continuous">
-      <parent link="${prefix}chassis_link"/>
-      <child link="${prefix}right_wheel"/>
-      <origin xyz="0 ${base_width/2} -${base_height/2}" rpy="0 0 ${PI/2}"/>
-      <axis xyz="1 0 0"/>
-      <limit effort="100.0" velocity="1.0"/>
-      <dynamics damping="0.2"/>
-    </joint>
     <!-- rear wheels -->
     <!-- rear right wheel -->
@@ -123,5 +87,4 @@
       <limit effort="100.0" velocity="1.0"/>
       <dynamics damping="0.2"/>
-      <mimic joint="${prefix}right_wheel_joint" multiplier="1.0" offset="0.0"/>
     </joint>
     <gazebo reference="${prefix}rear_right_wheel">
@@ -159,5 +122,4 @@
       <limit effort="100.0" velocity="1.0"/>
       <dynamics damping="0.2"/>
-      <mimic joint="${prefix}left_wheel_joint" multiplier="1.0" offset="0.0"/>
     </joint>
     <gazebo reference="${prefix}rear_left_wheel">
@@ -196,5 +158,4 @@
       <limit effort="100.0" velocity="1.0"/>
       <dynamics damping="0.2"/>
-      <mimic joint="${prefix}right_wheel_joint" multiplier="1.0" offset="0.0"/>
     </joint>
     <gazebo reference="${prefix}front_right_wheel">
@@ -232,5 +193,4 @@
       <limit effort="100.0" velocity="1.0"/>
       <dynamics damping="0.2"/>
-      <mimic joint="${prefix}left_wheel_joint" multiplier="1.0" offset="0.0"/>
     </joint>
     <gazebo reference="${prefix}front_left_wheel">

Commit message: fix URDF and prepare to slamtoolbox

File: description/ros2_control/hoverboard_driver.ros2_control.xacro (robot description, xacro)
@@ -6,6 +6,6 @@
         <plugin>hoverboard_driver/hoverboard_driver</plugin>
         <param name="prefix">${prefix}</param>
-        <param name="wheel_radius">0.0825</param>
-        <param name="max_velocity">1.0</param>
+        <param name="wheel_radius">0.085</param>
+        <param name="max_velocity">2.0</param>
         <param name="device">${device}</param>
       </hardware>

File: description/urdf/diffbot_description.urdf.xacro (robot description, xacro)
@@ -5,11 +5,12 @@
   <xacro:property name="PI" value="3.1415926535897931"/>
   <xacro:property name="base_mass" value="4.0" /> <!-- arbitrary value for base mass -->
-  <xacro:property name="base_width" value="0.260" />
-  <xacro:property name="base_length" value="0.525" />
-  <xacro:property name="base_height" value="0.060" />
-  <xacro:property name="wheelbase" value="0.325" />
+  <xacro:property name="base_width" value="0.465" />
+  <xacro:property name="base_length" value="0.760" />
+  <xacro:property name="base_height" value="0.040" />
+  <xacro:property name="wheelbase" value="0.320" />
   <xacro:property name="wheel_mass" value="0.34055" /> <!-- arbitrary value for wheel mass -->
-  <xacro:property name="wheel_len" value="0.045" />
-  <xacro:property name="wheel_radius" value="0.05" />
+  <xacro:property name="wheel_len" value="0.060" />
+  <xacro:property name="wheel_seperate" value="0.520"/>
+  <xacro:property name="wheel_radius" value="0.085" />
   <xacro:property name="lidar_height" value="0.05" />
   <xacro:property name="lidar_radius" value="0.03" />
@@ -17,8 +18,12 @@
   <!-- Base Link -->
   <link name="${prefix}base_link" />
-    <!-- <joint name= "base-chassis">
-    <parent link="${prefix}base_link"/>
-    <child link="${prefix}chassis_link"/>
-    <joint/> -->
+  <!-- Base Footprint Link-->
+  <link name="base_footprint">
+  </link>
+  <joint name="base_footprint_joint" type = "fixed">
+    <parent link="base_link"/>
+    <child link="base_footprint"/>
+    <origin xyz="0 0 0" rpy= "0 0 0"/>
+  </joint>
   <!-- Chassis -->
   <link name="${prefix}chassis_link">
@@ -43,6 +48,6 @@
           iyy="0.000270" iyz="0.0"
           izz="0.000426"/>
-      </inertial>
-    </link>
+    </inertial>
+  </link>
     <joint name="${prefix}chassis_joint" type="fixed">
       <parent link="${prefix}base_link"/>
@@ -83,5 +88,5 @@
       <parent link="${prefix}chassis_link"/>
       <child link="${prefix}rear_right_wheel"/>
-      <origin xyz="-${wheelbase/2} ${base_width/2} -${base_height/2}" rpy="0 0 ${PI/2}"/>
+      <origin xyz="-${wheelbase/2} ${wheel_seperate/2} -${base_height/2}" rpy="0 0 ${PI/2}"/>
       <axis xyz="1 0 0"/>
       <limit effort="100.0" velocity="1.0"/>
@@ -118,5 +123,5 @@
       <parent link="${prefix}chassis_link" />
       <child link="${prefix}rear_left_wheel" />
-      <origin xyz="-${wheelbase/2} -${base_width/2} -${base_height/2}" rpy="0 0 ${PI/2}"/>
+      <origin xyz="-${wheelbase/2} -${wheel_seperate/2} -${base_height/2}" rpy="0 0 ${PI/2}"/>
       <axis xyz="1 0 0"/>
       <limit effort="100.0" velocity="1.0"/>
@@ -154,5 +159,5 @@
       <parent link="${prefix}chassis_link" />
       <child link="${prefix}front_right_wheel" />
-      <origin xyz="${wheelbase/2} ${base_width/2} -${base_height/2}" rpy="0 0 ${PI/2}"/>
+      <origin xyz="${wheelbase/2} ${wheel_seperate/2} -${base_height/2}" rpy="0 0 ${PI/2}"/>
       <axis xyz="1 0 0"/>
       <limit effort="100.0" velocity="1.0"/>
@@ -189,5 +194,5 @@
       <parent link="${prefix}chassis_link" />
       <child link="${prefix}front_left_wheel" />
-      <origin xyz="${wheelbase/2} -${base_width/2} -${base_height/2}" rpy="0 0 ${PI/2}"/>
+      <origin xyz="${wheelbase/2} -${wheel_seperate/2} -${base_height/2}" rpy="0 0 ${PI/2}"/>
       <axis xyz="1 0 0"/>
       <limit effort="100.0" velocity="1.0"/>

Commit message: change steer function and debug controller odom

File: description/ros2_control/hoverboard_driver.ros2_control.xacro (robot description, xacro)
@@ -9,4 +9,5 @@
         <param name="max_velocity">2.0</param>
         <param name="device">${device}</param>
+        <param name="wheel_base">0.32</param>
       </hardware>
       <joint name="${prefix}left_wheel_joint">

File: description/urdf/diffbot_description.urdf.xacro (robot description, xacro)
@@ -9,5 +9,5 @@
   <xacro:property name="base_height" value="0.040" />
   <xacro:property name="wheelbase" value="0.320" />
-  <xacro:property name="wheel_mass" value="0.34055" /> <!-- arbitrary value for wheel mass -->
+  <xacro:property name="wheel_mass" value="1.0" /> <!-- arbitrary value for wheel mass -->
   <xacro:property name="wheel_len" value="0.060" />
   <xacro:property name="wheel_seperate" value="0.520"/>

Commit message: macth real rpm and cmd rpm

File: description/ros2_control/hoverboard_driver.ros2_control.xacro (robot description, xacro)
@@ -9,5 +9,5 @@
         <param name="max_velocity">2.0</param>
         <param name="device">${device}</param>
-        <param name="wheel_base">0.32</param>
+        <param name="wheel_separation">0.52</param>
       </hardware>
       <joint name="${prefix}left_wheel_joint">

File: description/urdf/diffbot_description.urdf.xacro (robot description, xacro)
@@ -11,5 +11,5 @@
   <xacro:property name="wheel_mass" value="1.0" /> <!-- arbitrary value for wheel mass -->
   <xacro:property name="wheel_len" value="0.060" />
-  <xacro:property name="wheel_seperate" value="0.520"/>
+  <xacro:property name="wheel_separation" value="0.520"/>
   <xacro:property name="wheel_radius" value="0.085" />
   <xacro:property name="lidar_height" value="0.05" />
@@ -88,5 +88,5 @@
       <parent link="${prefix}chassis_link"/>
       <child link="${prefix}rear_right_wheel"/>
-      <origin xyz="-${wheelbase/2} -${wheel_seperate/2} -${base_height/2}" rpy="0 0 ${PI/2}"/>
+      <origin xyz="-${wheelbase/2} -${wheel_separation/2} -${base_height/2}" rpy="0 0 ${PI/2}"/>
       <axis xyz="1 0 0"/>
       <limit effort="100.0" velocity="1.0"/>
@@ -123,5 +123,5 @@
       <parent link="${prefix}chassis_link" />
       <child link="${prefix}rear_left_wheel" />
-      <origin xyz="-${wheelbase/2} ${wheel_seperate/2} -${base_height/2}" rpy="0 0 ${PI/2}"/>
+      <origin xyz="-${wheelbase/2} ${wheel_separation/2} -${base_height/2}" rpy="0 0 ${PI/2}"/>
       <axis xyz="1 0 0"/>
       <limit effort="100.0" velocity="1.0"/>
@@ -159,5 +159,5 @@
       <parent link="${prefix}chassis_link" />
       <child link="${prefix}front_right_wheel" />
-      <origin xyz="${wheelbase/2} -${wheel_seperate/2} -${base_height/2}" rpy="0 0 ${PI/2}"/>
+      <origin xyz="${wheelbase/2} -${wheel_separation/2} -${base_height/2}" rpy="0 0 ${PI/2}"/>
       <axis xyz="1 0 0"/>
       <limit effort="100.0" velocity="1.0"/>
@@ -194,5 +194,5 @@
       <parent link="${prefix}chassis_link" />
       <child link="${prefix}front_left_wheel" />
-      <origin xyz="${wheelbase/2} ${wheel_seperate/2} -${base_height/2}" rpy="0 0 ${PI/2}"/>
+      <origin xyz="${wheelbase/2} ${wheel_separation/2} -${base_height/2}" rpy="0 0 ${PI/2}"/>
       <axis xyz="1 0 0"/>
       <limit effort="100.0" velocity="1.0"/>
