Commit message: fix rviz tf error

File: description/urdf/diffbot_description.urdf.xacro (robot description, xacro)
@@ -226,9 +226,9 @@
       <origin xyz="0 0 ${base_height/2}" rpy="0 0 0"/>
     </joint>
-    <gazebo reference="${prefix}lidar_sensor">
+    <gazebo reference="${prefix}laser">
         <material>Gazebo/Black</material>
     </gazebo>
     <!-- LiDAR Sensor -->
-    <link name="${prefix}lidar_sensor">
+    <link name="${prefix}laser">
       <visual>
         <origin xyz="0 0 0" rpy="0 0 0"/>
@@ -244,16 +244,8 @@
         </geometry>
       </collision>
-      <inertial>
-        <origin xyz="0 0 0" rpy="0 0 0"/>
-        <mass value="0.01"/>
-        <inertia
-          ixx="0.000270" ixy="0.0" ixz="0.0"
-          iyy="0.000270" iyz="0.0"
-          izz="0.000426"/>
-      </inertial>
-    </link>
-    <joint name="${prefix}lidar_joint" type="fixed">
+    </link>
+    <joint name="${prefix}laser_joint" type="fixed">
       <parent link="${prefix}chassis_link"/>
-      <child link="${prefix}lidar_sensor"/>
+      <child link="${prefix}laser"/>
       <origin xyz="0 0 ${base_height/2 + lidar_height/2}" rpy="0 0 0"/>
     </joint>

Commit message: change encoder TICKS_PER_RROTATION

File: description/urdf/diffbot_description.urdf.xacro (robot description, xacro)
@@ -4,5 +4,5 @@
   <!-- Constants for robot dimensions -->
   <xacro:property name="PI" value="3.1415926535897931"/>
-  <xacro:property name="base_mass" value="4.0" /> <!-- arbitrary value for base mass -->
+  <xacro:property name="base_mass" value="10.0" /> <!-- arbitrary value for base mass -->
   <xacro:property name="base_width" value="0.465" />
   <xacro:property name="base_length" value="0.760" />

Commit message: add lidar pkg and inital pose

File: description/urdf/diffbot_description.urdf.xacro (robot description, xacro)
@@ -19,11 +19,11 @@
   <link name="${prefix}base_link" />
   <!-- Base Footprint Link-->
-  <link name="base_footprint">
-  </link>
-  <joint name="base_footprint_joint" type = "fixed">
+  <!-- <link name="base_footprint">
+  </link> -->
+  <!-- <joint name="base_footprint_joint" type = "fixed">
     <parent link="base_link"/>
     <child link="base_footprint"/>
     <origin xyz="0 0 0" rpy= "0 0 0"/>
-  </joint>
+  </joint> -->
   <!-- Chassis -->
   <link name="${prefix}chassis_link">
@@ -88,5 +88,5 @@
       <parent link="${prefix}chassis_link"/>
       <child link="${prefix}rear_right_wheel"/>
-      <origin xyz="-${wheelbase/2} ${wheel_seperate/2} -${base_height/2}" rpy="0 0 ${PI/2}"/>
+      <origin xyz="-${wheelbase/2} -${wheel_seperate/2} -${base_height/2}" rpy="0 0 ${PI/2}"/>
       <axis xyz="1 0 0"/>
       <limit effort="100.0" velocity="1.0"/>
@@ -123,5 +123,5 @@
       <parent link="${prefix}chassis_link" />
       <child link="${prefix}rear_left_wheel" />
-      <origin xyz="-${wheelbase/2} -${wheel_seperate/2} -${base_height/2}" rpy="0 0 ${PI/2}"/>
+      <origin xyz="-${wheelbase/2} ${wheel_seperate/2} -${base_height/2}" rpy="0 0 ${PI/2}"/>
       <axis xyz="1 0 0"/>
       <limit effort="100.0" velocity="1.0"/>
@@ -159,5 +159,5 @@
       <parent link="${prefix}chassis_link" />
       <child link="${prefix}front_right_wheel" />
-      <origin xyz="${wheelbase/2} ${wheel_seperate/2} -${base_height/2}" rpy="0 0 ${PI/2}"/>
+      <origin xyz="${wheelbase/2} -${wheel_seperate/2} -${base_height/2}" rpy="0 0 ${PI/2}"/>
       <axis xyz="1 0 0"/>
       <limit effort="100.0" velocity="1.0"/>
@@ -194,5 +194,5 @@
       <parent link="${prefix}chassis_link" />
       <child link="${prefix}front_left_wheel" />
-      <origin xyz="${wheelbase/2} -${wheel_seperate/2} -${base_height/2}" rpy="0 0 ${PI/2}"/>
+      <origin xyz="${wheelbase/2} ${wheel_seperate/2} -${base_height/2}" rpy="0 0 ${PI/2}"/>
       <axis xyz="1 0 0"/>
       <limit effort="100.0" velocity="1.0"/>
@@ -253,5 +253,5 @@
       <parent link="${prefix}chassis_link"/>
       <child link="${prefix}laser"/>
-      <origin xyz="0 0 ${base_height/2 + lidar_height/2}" rpy="0 0 0"/>
+      <origin xyz="0 0 ${base_height/2 + lidar_height/2}" rpy="${PI} 0 ${PI}"/>
     </joint>
     <!-- <xacro:include filename="lidar.xacro"/>

Commit message: IMU position adjustment

File: description/urdf/diffbot_description.urdf.xacro (robot description, xacro)
@@ -229,5 +229,5 @@
       <parent link="${prefix}chassis_link"/>
       <child link="${prefix}imu_sensor"/>
-      <origin xyz="0 0 ${base_height/2}" rpy="0 0 0"/>
+      <origin xyz="0.12 0 ${base_height/2}" rpy="0 0 0"/>
     </joint>
     <gazebo reference="${prefix}laser">

Commit message: Update URDF file for version_white

File: description/urdf/diffbot_description.urdf.xacro (robot description, xacro)
@@ -5,8 +5,8 @@
   <xacro:property name="PI" value="3.1415926535897931"/>
   <xacro:property name="base_mass" value="10.0" /> <!-- arbitrary value for base mass -->
-  <xacro:property name="base_width" value="0.465" />
-  <xacro:property name="base_length" value="0.760" />
-  <xacro:property name="base_height" value="0.040" />
-  <xacro:property name="wheelbase" value="0.320" />
+  <xacro:property name="base_width" value="0.635" />
+  <xacro:property name="base_length" value="0.880" />
+  <xacro:property name="base_height" value="0.16" />
+  <xacro:property name="wheelbase" value="0.470" />
   <xacro:property name="wheel_mass" value="1.0" /> <!-- arbitrary value for wheel mass -->
   <xacro:property name="wheel_len" value="0.060" />
