Commit message: version_white and ydlidar x4

File: description/urdf/diffbot.urdf.xacro (robot description, xacro)
@@ -9,5 +9,5 @@
   <xacro:include filename="$(find hoverboard_driver)/ros2_control/hoverboard_driver.ros2_control.xacro"/>
   <xacro:diffbot prefix="$(arg prefix)" />
-  <xacro:hoverboard_driver_ros2_control name="front_hoverboard" prefix="front_" device="/dev/ttyUSB0"/>
-  <xacro:hoverboard_driver_ros2_control name="rear_hoverboard" prefix="rear_" device="/dev/ttyUSB1"/>
+  <xacro:hoverboard_driver_ros2_control name="front_hoverboard" prefix="front_" device="/dev/front_wheel"/>
+  <xacro:hoverboard_driver_ros2_control name="rear_hoverboard" prefix="rear_" device="/dev/rear_wheel"/>
 </robot>

File: description/urdf/diffbot_description.urdf.xacro (robot description, xacro)
@@ -235,5 +235,5 @@
     </gazebo>
     <!-- LiDAR Sensor -->
-    <link name="${prefix}laser">
+    <link name="${prefix}laser_frame">
       <visual>
         <origin xyz="0 0 0" rpy="0 0 0"/>
@@ -252,6 +252,6 @@
     <joint name="${prefix}laser_joint" type="fixed">
       <parent link="${prefix}chassis_link"/>
-      <child link="${prefix}laser"/>
-      <origin xyz="0 0 ${base_height/2 + lidar_height/2}" rpy="${PI} 0 ${PI}"/>
+      <child link="${prefix}laser_frame"/>
+      <origin xyz="0 0 ${base_height/2 + lidar_height/2}" rpy="0 0 0"/>
     </joint>
     <!-- <xacro:include filename="lidar.xacro"/>
